Commit message: fix(stack): EKF drift, QoS mismatch, Nav2 plugins, URDF wheels, RC deadzone
Foxglove vizualizáció és teljes stack stabilizálás:

- EKF: publish_tf=false, controller enable_odom_tf=true — egyetlen szenzor
  (wheel odom) mellett az EKF random walk driftet okozott. Controller adja
  az odom→base_link TF-et amíg IMU nincs konfigurálva.
- EKF: odom topic /odom → /diff_drive_controller/odom (helyes topic név)
- EKF: IMU kikommentezve (kamera frame ≠ robot frame, -66° roll)
- EKF: process noise 0.05→0.001 (IMU visszakapcsoláskor növelendő)
- QoS: safety_supervisor + startup_supervisor IMU sub SensorDataQoS()
  (RealSense BEST_EFFORT-tel publikál, RELIABLE sub nem kap adatot)
- Nav2: összes plugin név / → :: (Jazzy requirement), plugin_lib_names
  eltávolítva (auto-register), SLAM bond_timeout workaround
- URDF: 4 kerék helyes pozícióban, front wheels mimic joints, helyes
  tengely orientáció (z=up, y=left, x=forward)
- RC teleop: deadzone paraméter (0.05) — joystick zaj nem driftel odomot
- .env: tilt check kikapcsolva (CHECK_TILT_ENABLED=false, 90° limitek)
- docker-compose: volume mount config/launch fájlokhoz (rebuild nélküli
  hot-reload)
- Makefile: agent-restart target (bridge session loss workaround)
- backlog: URDF mesh, IMU frame, slam lifecycle, controller jitter

Co-Authored-By: Claude Opus 4.6 <noreply@anthropic.com>

File: robot_description/urdf/robot.urdf.xacro (robot description, xacro)
@@ -93,11 +93,13 @@
   <!-- ============================================================
        WHEEL MACRO
-       rpy="${-pi/2} 0 0" rotates the cylinder so its geometric axis
-       aligns with the robot Y axis (lateral), which is the correct
-       spin axis for diff_drive_controller with axis xyz="0 0 1".
+       Joint frame: x=forward, y=left, z=up (ROS convention).
+       Spin axis = Y (lateral) → axis xyz="0 1 0".
+       Cylinder visual is rotated 90° so its geometric axis aligns
+       with the Y (spin) axis.
        ============================================================ -->
   <xacro:macro name="wheel" params="name x y">
     <link name="${name}">
       <visual>
+        <origin xyz="0 0 0" rpy="${pi/2} 0 0"/>
         <geometry>
           <cylinder radius="${wheel_radius}" length="${wheel_width}"/>
@@ -105,4 +107,5 @@
       </visual>
       <collision>
+        <origin xyz="0 0 0" rpy="${pi/2} 0 0"/>
         <geometry>
           <cylinder radius="${wheel_radius}" length="${wheel_width}"/>
@@ -114,6 +117,6 @@
       <parent link="base_link"/>
       <child  link="${name}"/>
-      <origin xyz="${x} ${y} ${wheel_radius}" rpy="${-pi/2} 0 0"/>
-      <axis   xyz="0 0 1"/>
+      <origin xyz="${x} ${y} ${wheel_radius}" rpy="0 0 0"/>
+      <axis   xyz="0 1 0"/>
     </joint>
   </xacro:macro>
@@ -143,7 +146,43 @@
   <xacro:wheel name="rear_left_wheel"   x="${-axle_offset}" y="${ wheel_separation / 2.0}"/>
   <xacro:wheel name="rear_right_wheel"  x="${-axle_offset}" y="${-wheel_separation / 2.0}"/>
-  <!-- Front — mechanically linked to rear (same chain/shaft per side) -->
-  <xacro:wheel name="front_left_wheel"  x="${ axle_offset}" y="${ wheel_separation / 2.0}"/>
-  <xacro:wheel name="front_right_wheel" x="${ axle_offset}" y="${-wheel_separation / 2.0}"/>
+  <!-- Front — mechanically linked to rear (same chain/shaft per side).
+       Mimic joints: robot_state_publisher mirrors rear wheel joint states
+       to front wheels automatically. No separate joint_state needed. -->
+  <link name="front_left_wheel">
+    <visual>
+      <origin xyz="0 0 0" rpy="${pi/2} 0 0"/>
+      <geometry><cylinder radius="${wheel_radius}" length="${wheel_width}"/></geometry>
+    </visual>
+    <collision>
+      <origin xyz="0 0 0" rpy="${pi/2} 0 0"/>
+      <geometry><cylinder radius="${wheel_radius}" length="${wheel_width}"/></geometry>
+    </collision>
+    <xacro:cylinder_inertia m="${wheel_mass}" r="${wheel_radius}" h="${wheel_width}"/>
+  </link>
+  <joint name="front_left_wheel_joint" type="continuous">
+    <parent link="base_link"/>
+    <child  link="front_left_wheel"/>
+    <origin xyz="${axle_offset} ${wheel_separation / 2.0} ${wheel_radius}" rpy="0 0 0"/>
+    <axis   xyz="0 1 0"/>
+    <mimic  joint="rear_left_wheel_joint" multiplier="1.0" offset="0.0"/>
+  </joint>
+  <link name="front_right_wheel">
+    <visual>
+      <origin xyz="0 0 0" rpy="${pi/2} 0 0"/>
+      <geometry><cylinder radius="${wheel_radius}" length="${wheel_width}"/></geometry>
+    </visual>
+    <collision>
+      <origin xyz="0 0 0" rpy="${pi/2} 0 0"/>
+      <geometry><cylinder radius="${wheel_radius}" length="${wheel_width}"/></geometry>
+    </collision>
+    <xacro:cylinder_inertia m="${wheel_mass}" r="${wheel_radius}" h="${wheel_width}"/>
+  </link>
+  <joint name="front_right_wheel_joint" type="continuous">
+    <parent link="base_link"/>
+    <child  link="front_right_wheel"/>
+    <origin xyz="${axle_offset} ${-wheel_separation / 2.0} ${wheel_radius}" rpy="0 0 0"/>
+    <axis   xyz="0 1 0"/>
+    <mimic  joint="rear_right_wheel_joint" multiplier="1.0" offset="0.0"/>
+  </joint>
   <!-- ============================================================
        LIDAR — RPLidar A2

Commit message: feat(description): STL meshes, valós méretek, Foxglove mesh szerver
- URDF frissítve valós méretekkel (Ø380mm kerék, 700mm nyomtáv, pontos chassis/platform méretek)
- STL mesh-ek hozzáadva (chassis, platform, wheel) primitív geometriák helyett
- mesh_server.py HTTP szerver Foxglove böngészős mesh betöltéshez
- Foxglove Dockerfile: ament package regisztráció + asset_uri_allowlist
- docker-compose: mesh volume mount-ok és mesh_server szolgáltatás
- twist_mux: /cmd_vel_foxglove topic (priority 30)

Co-Authored-By: Claude Opus 4.6 (1M context) <noreply@anthropic.com>

File: robot_description/urdf/robot.urdf.xacro (robot description, xacro)
@@ -2,10 +2,15 @@
 <!--
   Talicska rover — robot_description
-  Physical measurements:
-    Chassis:        1100 × 800 mm, ~350 mm tall
-    Wheels:         Ø400 mm (r=0.2m), 150 mm wide, 800 mm track
-    Axles:          ±235 mm from rotation centre (= base_link)
-    base_link:      rotation centre, at ground plane (z=0)
-    Tilt hinge:     300 mm from platform front → 205 mm forward of base_link
+  Physical measurements (2026-03-16, verified):
+    Vehicle:        1100 mm long, 800 mm wide (wheel edge to edge), 750 mm tall
+    Chassis:        640 × 550 × 140 mm, bottom at 120 mm, top at 260 mm
+    Wheels:         Ø380 mm (r=190mm), 100 mm wide, 700 mm track (centre-centre)
+    Axles:          front 340 mm from vehicle front, rear 790 mm → ±225 mm from base_link
+    base_link:      rotation centre (axle midpoint), 565 mm from vehicle front, at ground (z=0)
+    Chassis front:  240 mm behind vehicle front → +325 mm from base_link
+    Platform:       1100 × 750 × 300 mm, bottom at 450 mm, tilts forward
+    Tilt hinge:     chassis top (260 mm), 20 mm from chassis front → +305 mm from base_link
+    LiDAR:          on chassis, 340 mm from chassis front → -15 mm from base_link, Z=295 mm
+    Camera:         chassis front edge, Z=290 mm (lens centre 30 mm above chassis top)
   Wheel naming convention:
     rear_left / rear_right   — driven by RoboClaw (ros2_control joints)
@@ -40,28 +45,46 @@
   <xacro:arg name="encoder_max_speed_rad_s"   default="30.0"/>
   <!-- ============================================================
+       MESH BASE URL
+       Foxglove needs HTTP access to meshes (package:// doesn't work in browser).
+       Override at launch: xacro robot.urdf.xacro mesh_base:=package://robot_description
+       Alternatives:
+         LAN:       http://192.168.68.122:8081/robot_description
+         Tailscale: http://100.71.242.128:8081/robot_description
+         Robot net: http://10.0.10.1:8081/robot_description
+       ============================================================ -->
+  <xacro:arg name="mesh_base" default="http://192.168.68.122:8081/robot_description"/>
+  <xacro:property name="mesh_base" value="$(arg mesh_base)"/>
+  <!-- ============================================================
        GEOMETRY CONSTANTS  (metres)
        ============================================================ -->
-  <!-- Chassis -->
-  <xacro:property name="chassis_length"    value="1.1"/>
-  <xacro:property name="chassis_width"     value="0.8"/>
-  <xacro:property name="chassis_height"    value="0.35"/>
-  <!-- base_link is 505 mm from front, 595 mm from rear.
-       Visual box origin is at the chassis geometric centre: -->
-  <xacro:property name="chassis_x_offset"  value="${0.505 - chassis_length / 2.0}"/> <!-- -0.045 m -->
+  <!-- Chassis (alváz) -->
+  <xacro:property name="chassis_length"    value="0.64"/>
+  <xacro:property name="chassis_width"     value="0.55"/>
+  <xacro:property name="chassis_height"    value="0.14"/>
+  <xacro:property name="chassis_bottom_z"  value="0.12"/>
+  <!-- Chassis centre in base_link frame:
+       chassis front = +0.325, rear = -0.315, centre = +0.005 -->
+  <xacro:property name="chassis_x_offset"  value="0.005"/>
+  <xacro:property name="chassis_z_centre"  value="${chassis_bottom_z + chassis_height / 2.0}"/> <!-- 0.19 m -->
   <!-- Wheels -->
-  <xacro:property name="wheel_radius"      value="0.2"/>
-  <xacro:property name="wheel_width"       value="0.15"/>
-  <xacro:property name="wheel_separation"  value="0.8"/>
-  <!-- Axles are equidistant from rotation centre: 595-360 = 235 mm -->
-  <xacro:property name="axle_offset"       value="0.235"/>
-  <!-- Tilt platform -->
-  <xacro:property name="platform_length"   value="1.03"/>
+  <xacro:property name="wheel_radius"      value="0.19"/>
+  <xacro:property name="wheel_width"       value="0.1"/>
+  <xacro:property name="wheel_separation"  value="0.7"/>
+  <xacro:property name="axle_offset"       value="0.225"/>
+  <!-- Tilt platform (felépítmény) -->
+  <xacro:property name="platform_length"   value="1.1"/>
   <xacro:property name="platform_width"    value="0.75"/>
-  <xacro:property name="platform_height"   value="0.04"/>
-  <!-- Hinge is 300 mm from platform front.  Joint frame origin = hinge.
-       Platform CG from hinge (child +X = forward):
-         (0.3 - 0.73) / 2 = -0.215 m  (mostly behind hinge) -->
-  <xacro:property name="hinge_x"           value="${0.505 - 0.3}"/>           <!-- 0.205 m -->
-  <xacro:property name="platform_cg_x"     value="${0.3 - platform_length / 2.0}"/> <!-- -0.215 m -->
+  <xacro:property name="platform_height"   value="0.3"/>
+  <!-- Hinge at chassis top, 20 mm from chassis front
+       chassis front = +0.325 → hinge_x = +0.305
+       Platform bottom at 450 mm, hinge at 260 mm → support rod height = 190 mm
+       Platform centre Z relative to hinge: 190 + 150 = 340 mm
+       Platform centre X relative to hinge: vehicle centre (0.0) is at -0.305 from hinge
+       Platform spans +0.535 to -0.565 from base_link → centre = -0.015
+       Relative to hinge: -0.015 - 0.305 = -0.320 -->
+  <xacro:property name="hinge_x"           value="0.305"/>
+  <xacro:property name="hinge_z"           value="0.26"/>
+  <xacro:property name="platform_cg_x"     value="-0.32"/>
+  <xacro:property name="platform_cg_z"     value="0.34"/>
   <!-- Mass distribution  (total ≈ 108 kg) -->
   <xacro:property name="chassis_mass"      value="84.0"/>
@@ -95,13 +118,13 @@
        Joint frame: x=forward, y=left, z=up (ROS convention).
        Spin axis = Y (lateral) → axis xyz="0 1 0".
-       Cylinder visual is rotated 90° so its geometric axis aligns
-       with the Y (spin) axis.
-       ============================================================ -->
-  <xacro:macro name="wheel" params="name x y">
+       Mesh origin = hub/axle mount point. Left wheels use mesh as-is,
+       right wheels mirror on Y axis (scale 1 -1 1).
+       ============================================================ -->
+  <xacro:macro name="wheel" params="name x y reflect">
     <link name="${name}">
       <visual>
-        <origin xyz="0 0 0" rpy="${pi/2} 0 0"/>
+        <origin xyz="0 0 0" rpy="0 0 ${pi}"/>
         <geometry>
-          <cylinder radius="${wheel_radius}" length="${wheel_width}"/>
+          <mesh filename="${mesh_base}/meshes/wheel.stl" scale="1 ${reflect} 1"/>
         </geometry>
       </visual>
@@ -122,15 +145,16 @@
   </xacro:macro>
   <!-- ============================================================
-       BASE LINK  (rotation centre, at ground plane)
+       BASE LINK  (rotation centre, at ground plane z=0)
        ============================================================ -->
   <link name="base_link">
     <visual>
-      <origin xyz="${chassis_x_offset} 0 ${wheel_radius + chassis_height / 2.0}" rpy="0 0 0"/>
-      <geometry>
-        <box size="${chassis_length} ${chassis_width} ${chassis_height}"/>
-      </geometry>
-    </visual>
-    <collision>
-      <origin xyz="${chassis_x_offset} 0 ${wheel_radius + chassis_height / 2.0}" rpy="0 0 0"/>
+      <!-- STL origin aligned to model nullpoint; lift to chassis_z_centre (0.19m) -->
+      <origin xyz="0 0 ${chassis_z_centre}" rpy="0 0 0"/>
+      <geometry>
+        <mesh filename="${mesh_base}/meshes/chassis.stl"/>
+      </geometry>
+    </visual>
+    <collision>
+      <origin xyz="${chassis_x_offset} 0 ${chassis_z_centre}" rpy="0 0 0"/>
       <geometry>
         <box size="${chassis_length} ${chassis_width} ${chassis_height}"/>
@@ -144,6 +168,6 @@
        ============================================================ -->
   <!-- Rear — driven by RoboClaw via ros2_control -->
-  <xacro:wheel name="rear_left_wheel"   x="${-axle_offset}" y="${ wheel_separation / 2.0}"/>
-  <xacro:wheel name="rear_right_wheel"  x="${-axle_offset}" y="${-wheel_separation / 2.0}"/>
+  <xacro:wheel name="rear_left_wheel"   x="${-axle_offset}" y="${ wheel_separation / 2.0}" reflect="1"/>
+  <xacro:wheel name="rear_right_wheel"  x="${-axle_offset}" y="${-wheel_separation / 2.0}" reflect="-1"/>
   <!-- Front — mechanically linked to rear (same chain/shaft per side).
        Mimic joints: robot_state_publisher mirrors rear wheel joint states
@@ -151,6 +175,8 @@
   <link name="front_left_wheel">
     <visual>
-      <origin xyz="0 0 0" rpy="${pi/2} 0 0"/>
-      <geometry><cylinder radius="${wheel_radius}" length="${wheel_width}"/></geometry>
+      <origin xyz="0 0 0" rpy="0 0 ${pi}"/>
+      <geometry>
+        <mesh filename="${mesh_base}/meshes/wheel.stl" scale="1 1 1"/>
+      </geometry>
     </visual>
     <collision>
@@ -169,6 +195,8 @@
   <link name="front_right_wheel">
     <visual>
-      <origin xyz="0 0 0" rpy="${pi/2} 0 0"/>
-      <geometry><cylinder radius="${wheel_radius}" length="${wheel_width}"/></geometry>
+      <origin xyz="0 0 0" rpy="0 0 ${pi}"/>
+      <geometry>
+        <mesh filename="${mesh_base}/meshes/wheel.stl" scale="1 -1 1"/>
+      </geometry>
     </visual>
     <collision>
@@ -187,6 +215,6 @@
   <!-- ============================================================
        LIDAR — RPLidar A2
-       Mounted on top of chassis, forward-centre.
-       NOTE: exact XY position to be verified with physical measurements.
+       On chassis, 340 mm from chassis front → X = -0.015 m from base_link
+       Z = chassis top (0.26) + sensor half-height (0.035)
        ============================================================ -->
   <link name="lidar_link">
@@ -205,11 +233,10 @@
     <parent link="base_link"/>
     <child  link="lidar_link"/>
-    <!-- Top of chassis (z = wheel_radius + chassis_height) + sensor half-height -->
-    <origin xyz="0.3 0 ${wheel_radius + chassis_height + 0.035}" rpy="0 0 0"/>
+    <origin xyz="-0.015 0 0.295" rpy="0 0 0"/>
   </joint>
   <!-- ============================================================
        CAMERA — RealSense D435i
-       Mounted on front face of chassis, centre height.
-       NOTE: exact position to be verified with physical measurements.
+       Chassis front edge (X = +0.325), lens centre 30 mm above chassis top
+       Z = 0.26 + 0.03 = 0.29
        ============================================================ -->
   <link name="camera_link">
@@ -228,21 +255,22 @@
     <parent link="base_link"/>
     <child  link="camera_link"/>
-    <origin xyz="0.505 0 ${wheel_radius + chassis_height / 2.0}" rpy="0 0 0"/>
-  </joint>
-  <!-- ============================================================
-       TILT PLATFORM
-       Hinge 300 mm from platform front → hinge at x=0.205 m from base_link.
-       Joint frame origin = hinge.  Child +X = forward.
-       Platform CG is 215 mm behind the hinge.
+    <origin xyz="0.325 0 0.29" rpy="0 0 0"/>
+  </joint>
+  <!-- ============================================================
+       TILT PLATFORM (felépítmény)
+       Hinge at chassis top (Z=0.26), 20 mm from chassis front (X=+0.305).
+       Platform 1100×750×300 mm, bottom at 450 mm when level.
+       Support rods lift platform 190 mm above hinge.
+       Platform centre relative to hinge: X=-0.32, Z=+0.34
+       Tilts forward (positive Y rotation = nose down), max 45°.
        ============================================================ -->
   <link name="tilt_platform_link">
     <visual>
-      <origin xyz="${platform_cg_x} 0 0" rpy="0 0 0"/>
-      <geometry>
-        <box size="${platform_length} ${platform_width} ${platform_height}"/>
-      </geometry>
-    </visual>
-    <collision>
-      <origin xyz="${platform_cg_x} 0 0" rpy="0 0 0"/>
+      <geometry>
+        <mesh filename="${mesh_base}/meshes/platform.stl"/>
+      </geometry>
+    </visual>
+    <collision>
+      <origin xyz="${platform_cg_x} 0 ${platform_cg_z}" rpy="0 0 0"/>
       <geometry>
         <box size="${platform_length} ${platform_width} ${platform_height}"/>
@@ -255,8 +283,7 @@
     <parent link="base_link"/>
     <child  link="tilt_platform_link"/>
-    <origin xyz="${hinge_x} 0 ${wheel_radius + chassis_height + platform_height / 2.0}"
-            rpy="0 0 0"/>
+    <origin xyz="${hinge_x} 0 ${hinge_z}" rpy="0 0 0"/>
     <axis   xyz="0 1 0"/>
-    <limit  lower="${-pi/4}" upper="${pi/4}" effort="500.0" velocity="0.5"/>
+    <limit  lower="0.0" upper="${pi/4}" effort="500.0" velocity="0.5"/>
   </joint>
   <!-- ============================================================

Commit message: feat(imu): BNO085 dedikált IMU integráció (i2c-7, 0x4B)
- Dockerfile: bno08x_ros2_driver COPY hozzáadva
- sensors.launch.py: bno08x_driver node, /imu → /sensors/imu/data remap
- safety.launch.py: /camera/camera/imu → /sensors/imu/data remap (C++ érintetlen)
- robot.urdf.xacro: imu_link + imu_joint (X=0, Y=0, Z=0.295 — LiDAR magasság)
- robot_params.yaml: bno08x_driver szekció, EKF imu0 bekapcs., process_noise
  frissítve, tilt_roll 25° / tilt_pitch 20°, enable_imu_watchdog: true,
  startup check_tilt_enabled: true
- controllers.yaml: enable_odom_tf: false (EKF veszi át az odom→base_link TF-et)

TODO: imu_joint rpy véglegesítése fizikai mérés után

Co-Authored-By: Claude Sonnet 4.6 <noreply@anthropic.com>

File: robot_description/urdf/robot.urdf.xacro (robot description, xacro)
@@ -268,4 +268,29 @@
     <child  link="camera_link"/>
     <origin xyz="0.325 0 0.29" rpy="0 0 0"/>
+  </joint>
+  <!-- ============================================================
+       IMU — BNO085 (GY-BM0085)
+       Dedikált 9-DOF IMU, I2C (i2c-7, 0x4B).
+       Pozíció: robot hossztengelyén középen, LiDAR magasságán (X=0, Y=0, Z=0.295).
+         X=0: tengelyközép (base_link origó)
+         Y=0: szimmetriatengelyen
+         Z=0.295: LiDAR magassága (lidar_joint Z)
+       TODO: rpy — az IMU chip X/Y/Z tengelyeinek base_link-hez képesti forgatása.
+             Helytelen rpy → EKF hibás orientáció-korrekció.
+       ============================================================ -->
+  <link name="imu_link">
+    <visual>
+      <geometry><box size="0.02 0.02 0.005"/></geometry>
+    </visual>
+    <inertial>
+      <mass value="0.003"/>
+      <inertia ixx="0.0000001" iyy="0.0000001" izz="0.0000001" ixy="0" ixz="0" iyz="0"/>
+    </inertial>
+  </link>
+  <joint name="imu_joint" type="fixed">
+    <parent link="base_link"/>
+    <child  link="imu_link"/>
+    <!-- xyz mérve (2026-03-26). rpy TODO: mérés után frissítendő! -->
+    <origin xyz="0.0 0.0 0.295" rpy="0 0 0"/>
   </joint>
   <!-- ============================================================
