Commit message: feat(zed): ZED 2i kamera integráció — irányalapú kamera orchestráció
ZED 2i sztereó kamera (előre néző) teljes integrációja a robot stackbe.
RealSense D435i (hátra néző) megtartva REAR_NAV módhoz.

Makefile:
- camera-fwd-up/down: ZED 2i container orchestráció (FOLLOW/SHUTTLE)
- camera-rear-up/down: RealSense container orchestráció (REAR_NAV)
- camera-up: ROBOT_MODE-alapú automatikus kamera indítás
- make up = prestart check → kamerák → fő stack
- backward-compat aliasok: realsense-up, realsense-down

camera_director.py (scripts/):
- /cmd_vel_raw figyelése → ZED vagy RealSense depth relay
- Előremenet → /camera/fwd/depth (ZED), hátramese → /camera/rear/depth (RealSense)
- Hisztérézis 0.02 m/s, bounce guard 500ms, cmd_vel timeout 2s → FWD fallback
- sensors.launch.py: FOLLOW/SHUTTLE/NAVIGATION módban indul

URDF: zed_camera_link + zed_camera_joint (z=0.18m mért, x=0.480m PLACEHOLDER)
robot_params.yaml: SHUTTLE profil ÚJ, DOCKING→REAR_NAV átnevezés, ZED watchdog szekció
Dockerfile.foxglove: zed_interfaces sparse checkout + colcon build (skeleton vizualizáció)
ros_readiness_check.py: ZED depth topic check FOLLOW/SHUTTLE módban (30s timeout)
prestart.sh: ZED USB vendor check (2b03), ROBOT_MODE-aware (REAR_NAV→optional)
robot.repos: zed-jetson repo hozzáadva
.env: ROBOT_MODE kommentek frissítve (DOCKING→REAR_NAV)
docs: progress.md Fázis 3c, backlog.md ZED backlog tételek, project_overview.md frissítve

Co-Authored-By: Claude Sonnet 4.6 <noreply@anthropic.com>

File: robot_description/urdf/robot.urdf.xacro (robot description, xacro)
@@ -248,5 +248,5 @@
   </joint>
   <!-- ============================================================
-       CAMERA — RealSense D435i
+       CAMERA — RealSense D435i (rear-facing / docking)
        Chassis front edge (X = +0.325), lens centre 30 mm above chassis top
        Z = 0.26 + 0.03 = 0.29
@@ -268,4 +268,34 @@
     <child  link="camera_link"/>
     <origin xyz="0.325 0 0.29" rpy="0 0 0"/>
+  </joint>
+  <!-- ============================================================
+       ZED 2i — előre néző sztereó kamera (FOLLOW / SHUTTLE mód)
+       Saját Docker containerben fut (zed-jetson/), topic-ok: /zed/zed_node/*
+       Mérések (2026-04-06):
+         z = 0.18 m (180 mm a robot base aljától — mért érték)
+         y = 0.0   (hosszanti szimmetriatengelyen — mért érték)
+         x = 0.480 m  *** PLACEHOLDER — mérés szükséges! ***
+                      (könnyen frissíthető: volume-mounted, rebuild nem kell)
+       ZED 2i fizikai méret: 175 × 33 × 30 mm
+       IMU: csatlakoztatva, topic-ok elérhetők, TF letiltva (publish_imu_tf: false)
+       ============================================================ -->
+  <link name="zed_camera_link">
+    <visual>
+      <geometry><box size="0.175 0.033 0.030"/></geometry>
+      <material name="dark_grey"><color rgba="0.2 0.2 0.2 1.0"/></material>
+    </visual>
+    <collision>
+      <geometry><box size="0.175 0.033 0.030"/></geometry>
+    </collision>
+    <inertial>
+      <mass value="0.165"/>
+      <inertia ixx="0.0001" ixy="0" ixz="0" iyy="0.0001" iyz="0" izz="0.0001"/>
+    </inertial>
+  </link>
+  <joint name="zed_camera_joint" type="fixed">
+    <parent link="base_link"/>
+    <child  link="zed_camera_link"/>
+    <!-- z=0.18m (mért), y=0.0 (szimmetriatengelyen), x=0.480m (PLACEHOLDER — mérés kell) -->
+    <origin xyz="0.480 0.0 0.18" rpy="0 0 0"/>
   </joint>
   <!-- ============================================================

Commit message: feat: ZED 2i kivezetése a rendszerből (szerviz, 2026-05-05)
Ideiglenes konfiguráció: RealSense D435i veszi át az elülső kamera szerepét.
Hátsó kamera nincs. A ZED-specifikus kód megmarad kommentben a visszaállításhoz.

Érintett változások:
- prestart.sh: ZED USB check kikapcsolva (volt: required_nav minden módban — BLOKKOLTA az indítást)
- camera_director.py: D435i FWD irányban → /camera/fwd/depth; REAR irányban nincs relay
- robot.urdf.xacro: zed_camera_link + zed_camera_joint eltávolítva (kommentben megőrizve)
- Makefile: camera-up minden módban csak RealSense-t indít; camera-fwd-up no-op
- robot_params.yaml: profil kommentek frissítve (ZED → D435i ideiglenes)
- ros_readiness_check.py, sensors.launch.py: kommentek frissítve
- backlog.md: ZED visszaállítás feladat + integráció szünetel státusz

Co-Authored-By: Claude Sonnet 4.6 <noreply@anthropic.com>

File: robot_description/urdf/robot.urdf.xacro (robot description, xacro)
@@ -248,7 +248,9 @@
   </joint>
   <!-- ============================================================
-       CAMERA — RealSense D435i (rear-facing / docking)
-       Chassis front edge (X = +0.325), lens centre 30 mm above chassis top
-       Z = 0.26 + 0.03 = 0.29
+       CAMERA — RealSense D435i
+       IDEIGLENES KONFIGURÁCIÓ (2026-05-05): ZED 2i szervizen van.
+       A D435i előre néző kameraként üzemel a ZED helyett.
+       Pozíció: x=0.325 (chassis front edge), z=0.29 (lens centre ~30mm above top)
+       Visszaállításkor: ZED 2i link+joint visszaállítandó (lásd backlog)
        ============================================================ -->
   <link name="camera_link">
@@ -269,15 +271,6 @@
     <origin xyz="0.325 0 0.29" rpy="0 0 0"/>
   </joint>
-  <!-- ============================================================
-       ZED 2i — előre néző sztereó kamera (FOLLOW / SHUTTLE mód)
-       Saját Docker containerben fut (zed-jetson/), topic-ok: /zed/zed_node/*
-       Mérések (2026-04-06):
-         z = 0.18 m (180 mm a robot base aljától — mért érték)
-         y = 0.0   (hosszanti szimmetriatengelyen — mért érték)
-         x = 0.480 m  *** PLACEHOLDER — mérés szükséges! ***
-                      (könnyen frissíthető: volume-mounted, rebuild nem kell)
-       ZED 2i fizikai méret: 175 × 33 × 30 mm
-       IMU: csatlakoztatva, topic-ok elérhetők, TF letiltva (publish_imu_tf: false)
-       ============================================================ -->
+  <!-- ZED 2i frame eltávolítva (2026-05-05) — kamera szervizen van.
+       Visszaállításkor a következő blokk kerül vissza:
   <link name="zed_camera_link">
     <visual>
@@ -285,7 +278,5 @@
       <material name="dark_grey"><color rgba="0.2 0.2 0.2 1.0"/></material>
     </visual>
-    <collision>
-      <geometry><box size="0.175 0.033 0.030"/></geometry>
-    </collision>
+    <collision><geometry><box size="0.175 0.033 0.030"/></geometry></collision>
     <inertial>
       <mass value="0.165"/>
@@ -296,7 +287,7 @@
     <parent link="base_link"/>
     <child  link="zed_camera_link"/>
-    <!-- z=0.18m (mért), y=0.0 (szimmetriatengelyen), x=0.480m (PLACEHOLDER — mérés kell) -->
-    <origin xyz="0.480 0.0 0.18" rpy="0 0 0"/>
-  </joint>
+    <origin xyz="0.480 0.0 0.18" rpy="0 0 0"/>   z=0.18m (mért), x=0.480m (PLACEHOLDER)
+  </joint>
+  -->
   <!-- ============================================================
        IMU — BNO085 (GY-BM0085)

Commit message: feat(safety): LiDAR proximity zóna — non-latching, clusteres szűrő, enable kapcsoló
- IMU és LiDAR URDF pozíciók validálva és korrigálva fizikai mérés alapján
- Proximity zóna: superstructure_circumradius_m + proximity_safety_margin_m runtime számítás
- Clusteres min_points szűrő (ceruza kalibráció: max 7pt → küszöb 10pt)
- Non-latching viselkedés: akadály elhagyásakor automatikus recovery, E-Stop nem szükséges
- proximity_enabled YAML kapcsoló: false esetén teljesen inaktív
- Foxglove marker: /safety/proximity_zone (zöld/piros)
- scan_self_filter_calibrate.py: tartóoszlop szögmaszk kalibráló script
- Docs: robot_architecture.md + systemstatus.md frissítve

Co-Authored-By: Claude Sonnet 4.6 <noreply@anthropic.com>

File: robot_description/urdf/robot.urdf.xacro (robot description, xacro)
@@ -11,5 +11,5 @@
     Platform:       1100 × 750 × 300 mm, bottom at 450 mm, tilts forward
     Tilt hinge:     chassis top (260 mm), 20 mm from chassis front → +305 mm from base_link
-    LiDAR:          on chassis, 340 mm from chassis front → -15 mm from base_link, Z=295 mm
+    LiDAR:          on chassis, 600 mm from robot front, 360 mm from chassis front → -35 mm from base_link, Z=430 mm
     Camera:         chassis front edge, Z=290 mm (lens centre 30 mm above chassis top)
   Wheel naming convention:
@@ -245,5 +245,5 @@
     <parent link="base_link"/>
     <child  link="lidar_link"/>
-    <origin xyz="-0.015 0 0.295" rpy="0 0 0"/>
+    <origin xyz="-0.035 0.0 0.430" rpy="0 0 0"/>
   </joint>
   <!-- ============================================================
@@ -293,10 +293,9 @@
        IMU — BNO085 (GY-BM0085)
        Dedikált 9-DOF IMU, I2C (i2c-7, 0x4B).
-       Pozíció: robot hossztengelyén középen, LiDAR magasságán (X=0, Y=0, Z=0.295).
-         X=0: tengelyközép (base_link origó)
+       Pozíció (2026-05-07): 700mm robot elejétől, chassis aljától 250mm, szimmetriatengelyen.
+         X=-0.135: 565mm (base_link a fronttól) - 700mm = -135mm
          Y=0: szimmetriatengelyen
-         Z=0.295: LiDAR magassága (lidar_joint Z)
-       TODO: rpy — az IMU chip X/Y/Z tengelyeinek base_link-hez képesti forgatása.
-             Helytelen rpy → EKF hibás orientáció-korrekció.
+         Z=0.370: chassis alja (120mm) + 250mm
+       rpy=0: chip face-up, X→előre = REP-103 natív, koordináta-transzformáció nem kell.
        ============================================================ -->
   <link name="imu_link">
@@ -312,6 +311,6 @@
     <parent link="base_link"/>
     <child  link="imu_link"/>
-    <!-- xyz mérve (2026-03-26). rpy TODO: mérés után frissítendő! -->
-    <origin xyz="0.0 0.0 0.295" rpy="0 0 0"/>
+    <!-- xyz mérve (2026-05-07): 700mm robot elejétől → x=-0.135 (base_link 565mm a fronttól), chassis aljától 250mm → z=0.370. rpy=0: chip face-up, X→előre = REP-103 natív. -->
+    <origin xyz="-0.135 0.0 0.370" rpy="0 0 0"/>
   </joint>
   <!-- ============================================================

Commit message: urdf: D435i végleges pozíció — mért koordináták (2026-05-09)
Előlap 270mm robot elejétől, 160mm chassis aljától, szimmetriatengelyen.
  x=0.2825 (565mm front − 270mm − 12.5mm félmélység)
  y=0.0
  z=0.28  (chassis alja 120mm + 160mm)
IDEIGLENES jelzés eltávolítva.

Co-Authored-By: Claude Sonnet 4.6 <noreply@anthropic.com>

File: robot_description/urdf/robot.urdf.xacro (robot description, xacro)
@@ -12,5 +12,5 @@
     Tilt hinge:     chassis top (260 mm), 20 mm from chassis front → +305 mm from base_link
     LiDAR:          on chassis, 600 mm from robot front, 360 mm from chassis front → -35 mm from base_link, Z=430 mm
-    Camera:         chassis front edge, Z=290 mm (lens centre 30 mm above chassis top)
+    Camera:         front face 270 mm from vehicle front → centre X=+0.2825 m; Z=280 mm (160 mm above chassis bottom)
   Wheel naming convention:
     rear_left / rear_right   — driven by RoboClaw (ros2_control joints)
@@ -248,9 +248,9 @@
   </joint>
   <!-- ============================================================
-       CAMERA — RealSense D435i
-       IDEIGLENES KONFIGURÁCIÓ (2026-05-05): ZED 2i szervizen van.
-       A D435i előre néző kameraként üzemel a ZED helyett.
-       Pozíció: x=0.325 (chassis front edge), z=0.29 (lens centre ~30mm above top)
-       Visszaállításkor: ZED 2i link+joint visszaállítandó (lásd backlog)
+       CAMERA — RealSense D435i (végleges pozíció, 2026-05-09)
+       Mért pozíció: előlap 270mm robot elejétől, 160mm chassis aljától, szimmetriatengelyen.
+         X=+0.2825: vehicle front (565mm) − 270mm előlap − 12.5mm félmélység
+         Y=0.0:     szimmetriatengelyen
+         Z=0.28:    chassis alja (120mm) + 160mm
        ============================================================ -->
   <link name="camera_link">
@@ -269,5 +269,5 @@
     <parent link="base_link"/>
     <child  link="camera_link"/>
-    <origin xyz="0.325 0 0.29" rpy="0 0 0"/>
+    <origin xyz="0.2825 0.0 0.28" rpy="0 0 0"/>
   </joint>
   <!-- ZED 2i frame eltávolítva (2026-05-05) — kamera szervizen van.

Commit message: fix(motion): kanyarodás-irány HW+URDF tisztázás + startup E-Stop fix
KANYARODÁS-IRÁNY (többlépcsős diagnózis lezárva):
A földi RC-teszten kiderült: a kanyarodás fordított (RC + Foxglove teleop). Az
asztali fázisban nem volt tesztelt. Három iterációval rendezve:

1) `invert_*_motor: false` próba (commit 995b4fc): a kanyarodás OK lett, de az
   előre/hátra megfordult. A `motor_sign_` SW invertálás SZIMMETRIKUSAN hat
   mindkét csatornán → a tank-drive matematika miatt linear.x ÉS angular.z
   egyszerre invertálódik → aszimmetrikus fizikai bekötés mellett sehogy nem
   lehet a két tengelyen egyidejűleg helyes.

2) HW motor pólus-csere (felhasználói): a "rossz oldali" motor kábel-polaritás
   cseréje. A built-in encoder a motor-tengelyen ül, polaritás-csere automatikusan
   invertálja az encodert is → Basicmicro closed-loop konzisztens, nincs
   PID-divergencia. A HW most már szimmetrikus.

3) URDF `<ros2_control>` joint sorrend csere: a Basicmicro M1/M2 csatornakábel
   a robot fizikai jobb/bal motorához van bekötve. A `roboclaw_hardware` plugin
   az URDF joint sorrend szerint rendel csatornát. Csere: `rear_right_wheel_joint`
   első (M1), `rear_left_wheel_joint` második (M2). Az URDF wheel-link y
   koordináták és a `controllers.yaml left_wheel_names` MEGMARADTAK — TF, RViz,
   costmap REP-103 konzisztens. A csere transzparens az RC ÉS autonómia felé,
   mert mindkettő a diff_drive_controller-en át megy.

Végleges konfig:
- HW: motor pólus-csere kész (szimmetrikus)
- URDF `<ros2_control>`: rear_right (M1) → rear_left (M2)
- `roboclaw_hardware.invert_*_motor: false, false`

Nav2 kalibrációs mérés (10° kontrollált forgatási teszt):
- BALRA cmd +0.3 × 600ms → Δyaw +7.55° (elméleti +10.31°)
- JOBBRA cmd -0.3 × 600ms → Δyaw -7.53° (elméleti -10.31°)
- Szimmetria BAL/JOBB: 1.003 (tökéletes)
- Visszatérési hiba: +0.02° (zero ODOM drift 15° forgatás után)
- Effektív arány: 73% (Basicmicro acc-rampolás miatt, Nav2 zárt hurokban kezeli)

E-STOP STARTUP FIX:
A `startup_supervisor.cpp` CHECK_ESTOP fázis korábban 30s után FAULT-olt, ha az
E-Stop AKTÍV volt induláskor — stack restart aktív E-Stop mellett beragadt FAULT-ban,
csak újabb ROS restart oldotta. Új viselkedés: bridge ONLINE elég a startup-passhoz,
az AKTÍV state-et a runtime `safety_supervisor` kezeli (ESTOP state, Priority 1).
Felengedéskor automatikusan IDLE/RC-ba megy — természetes E-Stop viselkedés.

Co-Authored-By: Claude Opus 4.7 (1M context) <noreply@anthropic.com>

File: robot_description/urdf/robot.urdf.xacro (robot description, xacro)
@@ -378,5 +378,13 @@
       <param name="invert_right_motor">$(arg invert_right_motor)</param>
     </hardware>
-    <joint name="rear_left_wheel_joint">
+    <!-- Joint sorrend = Basicmicro motor csatornaallokáció:
+         joint[0] → M1, joint[1] → M2 (roboclaw_hardware plugin info_.joints[i] sorrend).
+         A fizikai kábelek: M1 csatlakozó → robot JOBB motor, M2 csatlakozó → robot BAL motor
+         (2026-05-12 földi RC-teszt diagnózis). Ezért a `rear_right_wheel_joint` az első
+         (M1), a `rear_left_wheel_joint` a második (M2). Az URDF link y koordináták és a
+         controllers.yaml `left_wheel_names: [rear_left_wheel_joint]` MEGMARADNAK — TF,
+         RViz, costmap helyesen REP-103 konzisztens. A csere transzparens az RC és
+         autonómia (Nav2/SLAM) felé. -->
+    <joint name="rear_right_wheel_joint">
       <command_interface name="velocity">
         <param name="min">-50</param>
@@ -386,5 +394,5 @@
       <state_interface name="velocity"/>
     </joint>
-    <joint name="rear_right_wheel_joint">
+    <joint name="rear_left_wheel_joint">
       <command_interface name="velocity">
         <param name="min">-50</param>

Commit message: feat(safety): /robot/mode Int32 sub + fizikai wheel paraméter kalibráció
A Pico E-Stop board 3-állású rotary kapcsoló (LEARN=0 / FOLLOW=1 / AUTO=2)
állapota nem érkezett meg a Jetson-ra. Gyökér ok: a safety_supervisor mode_sub_
std_msgs/String-ként deklarálta a /robot/mode topicot, miközben a Pico-firmware
Int32-t publikál (apps/estop/src/mode.c, MSG_INT32). DDS-szintű típus-mismatch
miatt a discovery nem kötötte össze publishert subscriberrel → 0 üzenet.

Fix:
- mode_sub_ típus: String → Int32, callback enum→String mapping
  (0=LEARN→"", 1=FOLLOW→"FOLLOW", 2=AUTO→"NAVIGATION")
- commanded_mode_ String használata változatlan a determine_state()-ben
- /safety/state JSON szerkezet érintetlen, /safety_parsed panelek működnek

Plus változtatások:
- wheel_separation: 0.7 → 0.72 (controllers.yaml + robot_params.yaml).
  Fizikailag mért 720 mm. 360°-os helyben-forgás teszt nem alkalmas (gumi-talaj
  slip ~33% dominál), fizikai mérőszalag a forrás.
- URDF wheel_radius: 0.19 → 0.1925 (fizikai 385 mm átmérő, csak vizualizációhoz).
  diff_drive_controller 0.19-en marad (kalibrált encoder_counts_per_rev: 144525-tel
  együtt 3 m fizikai = 3.012 m EKF, 0.4%).

BNO085 IMU yaw scale-bias 3 mérés átlaga -0.35% ±1% szórással — fixed scaling
nem stabil. yaw_scale_factor: 1.0 marad. EKF visszaállva yaw+vyaw módra
(chip-fusion stabilabb mint vyaw-only integráció).

SLAM mapping validálva (map3.png): loop closure detektálva, falak egyenesek
— autonóm navigációra kész.

Co-Authored-By: Claude Opus 4.7 (1M context) <noreply@anthropic.com>

File: robot_description/urdf/robot.urdf.xacro (robot description, xacro)
@@ -85,6 +85,15 @@
   <xacro:property name="chassis_z_centre"  value="${chassis_bottom_z + chassis_height / 2.0}"/> <!-- 0.19 m -->
   <!-- Wheels -->
-  <xacro:property name="wheel_radius"      value="0.19"/>
+  <!-- wheel_radius: fizikailag mért 385 mm átmérő (2026-05-12) → 0.1925 m sugár.
+       FIGYELEM: a `diff_drive_controller` (controllers.yaml + robot_params.yaml)
+       szándékosan 0.19 m-en marad, mert az `encoder_counts_per_rev: 144525`
+       kalibráció erre lett behangolva (3 m fizikai = 3.012 m EKF, 0.4% hiba).
+       Az URDF érték CSAK a robot_state_publisher TF-kozmetikát befolyásolja
+       (Foxglove vizualizáció), a diff_drive kinematika nem olvas innen. -->
+  <xacro:property name="wheel_radius"      value="0.1925"/>
   <xacro:property name="wheel_width"       value="0.1"/>
+  <!-- wheel_separation: kerék-közép → kerék-közép Y-irányban.
+       2026-05-12: visszaállítva 0.7-re az eredeti referenciára, friss
+       360°-os kalibrációs mérés folyamatban (pontosabb wheel-slip kompenzációval). -->
   <xacro:property name="wheel_separation"  value="0.7"/>
   <xacro:property name="axle_offset"       value="0.225"/>
